Commit message: Fix xacro expression and teleop executable
Use valid xacro conditional expressions for rotor fields and make teleop_keyboard.py executable so ros2 run can discover it.

File: src/drone_description/urdf/drone.urdf.xacro (robot description, xacro)
@@ -86,5 +86,5 @@
       <parent link="base_link"/>
       <child  link="${name}_arm"/>
-      <origin xyz="0 0 0" rpy="0 0 ${cw == 1 ? 0.785398 : -0.785398 + PI}"/>
+      <origin xyz="0 0 0" rpy="0 0 ${0.785398 if cw == 1 else -0.785398 + PI}"/>
     </joint>
     <!-- Rotor hub -->
@@ -95,5 +95,5 @@
           <cylinder radius="${rotor_radius}" length="${rotor_height}"/>
         </geometry>
-        <material name="${cw == 1 ? 'orange' : 'blue'}"/>
+        <material name="${'orange' if cw == 1 else 'blue'}"/>
       </visual>
       <inertial>
